File: EnviroLind.kicad_pcb (KiCad board)
At the start: 4 copper layers, 40.7 x 31.2 mm, 63 parts, among them J1 USB_C_Receptacle_USB2.0_16P, J2 qwiic, J3 Battery, Q1 AO3401A, SW3 Boot, SW4 User, U1 MCP73831-2-OT, U2 USBLC6-2P6, U3 AP2112K-3.3, U4 AP2112K-1.2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

Commit message: Start of power rework
Parts:
- added L1: 1µH, Inductor_SMD:L_0805_2012Metric, F.Cu at (85.7, 106.9)
- added R16: 51k, Resistor_SMD:R_0402_1005Metric, F.Cu at (110.7, 111.8)
- added R17: 511k, Resistor_SMD:R_0402_1005Metric, F.Cu at (88.0, 105.2)
- added R18: 91k, Resistor_SMD:R_0402_1005Metric, F.Cu at (90.0, 105.6)
- added R19: 1k, Resistor_SMD:R_0402_1005Metric, F.Cu at (88.0, 108.7)
- added R20: 1k, Resistor_SMD:R_0402_1005Metric, F.Cu at (90.0, 107.5)
- C1: value 4.7µF -> 22µF
- C2: value 4.7µF -> 47µF
- C3, C4: value 4.7µF -> 1µF
- U3: value AP2112K-3.3 -> TPS631000; footprint Package_TO_SOT_SMD:SOT-23-5 -> Package_TO_SOT_SMD:SOT-583-8
- U4: value AP2112K-1.2 -> TLV75512PDBV
- moved C2 5.35 mm to (89.7, 103.9), turned to 0 degrees
- moved R15 5.04 mm to (105.7, 112.8), turned to 0 degrees
- moved U7 4.45 mm to (86.0, 95.7), turned to 0 degrees
- moved R7 4.22 mm to (88.4, 95.0), turned to 180 degrees
- moved C7 3.79 mm to (85.5, 97.4), turned to 180 degrees
- moved Y1 2.45 mm to (89.5, 100.6)
- moved R8 2.44 mm to (88.4, 96.3), turned to 180 degrees
- moved C11 1.29 mm to (91.1, 99.8)
- moved C9 1.29 mm to (91.1, 101.7)
- moved D9 0.91 mm to (105.3, 111.6), turned to 180 degrees
- moved U3 0.36 mm to (88.0, 106.9), turned to 0 degrees
- moved C1 0.18 mm to (89.7, 110.6)
Connections:
- Q1 pad 1: +5V -> Net-(Q1-G)
- U3 pad 1: VCC -> +3.3V
- U3 pad 2: GND -> /LX2
- U3 pad 3: VCC -> /LX1
- U3 pad 4: unconnected-(U3-NC-Pad4) -> VCC
- U3 pad 5: +3.3V -> Net-(U3-EN)
- U4 pad 3: VCC -> LDO_EN
- U8 pad 27: unconnected-(U8-GPIO2/ADC1_CH2-Pad27) -> LDO_EN
Routing:
- net LDO_EN: track 0.00 -> 15.6 mm, vias 0 -> 2
- net SDA: track 12.9 -> 24.4 mm, vias 0 -> 2
- net SCL: track 12.4 -> 23.7 mm, vias 0 -> 2
- net VCC: track 50.0 -> 43.5 mm, vias 3 -> 5
- net +3.3V: track 23.5 -> 20.5 mm, vias 12 -> 13
- net GND: track 12.1 -> 14.9 mm, vias 56 -> 71
- net Net-(U3-FB): track 0.00 -> 2.74 mm
- net Net-(U3-Mode): track 0.00 -> 1.57 mm
- net Net-(Q1-G): track 0.00 -> 1.45 mm
- net Net-(U3-EN): track 0.00 -> 1.14 mm
- net XTAL_N: track 4.55 -> 3.72 mm
- net RX: track 3.47 -> 2.84 mm
- net BUTTON: track 23.2 -> 23.8 mm
- net XTAL_P: track 3.73 -> 4.27 mm
- net +5V: track 39.9 -> 39.7 mm, vias 5 -> 8
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- added copper zone on F.Cu, net +3.3V
- added copper zone on F.Cu, net /LX1
- added copper zone on F.Cu, net /LX2
- added copper zone on F.Cu, net VCC
