File: EnviroLind.kicad_sch (KiCad schematic)
At the start: 64 parts, among them J1 USB_C_Receptacle_USB2.0_16P, J2 qwiic, J3 Battery, Q1 AO3401A, SW2 Reset, SW3 Boot, SW4 User, U1 MCP73831-2-OT, U2 USBLC6-2P6, U3 AP2112K-3.3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

Commit message: Start of power rework
Parts:
- removed C8: 100n, Capacitor_SMD:C_0402_1005Metric, symbol Device:C
- removed U3: AP2112K-3.3, Package_TO_SOT_SMD:SOT-23-5, symbol Regulator_Linear:AP2112K-3.3
- removed U4: AP2112K-1.2, Package_TO_SOT_SMD:SOT-23-5, symbol Regulator_Linear:AP2112K-1.2
- removed U6: ENS161, LGA9:LGA9, symbol ENS161:ENS161
- added L1: 1µH, Inductor_SMD:L_0805_2012Metric, symbol Device:L
- added R16: 51k, Resistor_SMD:R_0402_1005Metric, symbol Device:R
- added R17: 511k, Resistor_SMD:R_0402_1005Metric, symbol Device:R
- added R18: 91k, Resistor_SMD:R_0402_1005Metric, symbol Device:R
- added R19, R20: 1k, Resistor_SMD:R_0402_1005Metric, symbol Device:R
- added U3: TPS631000, Package_TO_SOT_SMD:SOT-583-8, symbol TPS631000:TPS631000
- added U4: TLV75512PDBV, Package_TO_SOT_SMD:SOT-23-5, symbol Regulator_Linear:TLV75512PDBV
- C1: value 4.7µF -> 22µF
- C2: value 4.7µF -> 47µF
- C3, C4: value 4.7µF -> 1µF
- U5: value BME280 -> BME690
Connections:
- net +3.3V: now also R17.1, U3.1 (VO)
- net +5V: now also R16.1; no longer Q1.1 (G)
- net GND: now also R18.1, R20.1, U3.7 (GND), U4.2 (GND)
- net VCC: now also R19.1, U3.4 (VI), U4.1 (IN), U4.3 (EN)
- net LDO_EN: now reaches U8.27 (GPIO2/ADC1_CH2)
- net +1V2 renamed +1V8
- net +1V8: now also U4.5 (OUT)
- new net: R20.2, U3.6 (Mode)
- new net: R17.2, R18.2, U3.8 (FB)
- new net: Q1.1 (G), R16.2
- new net: R19.2, U3.5 (EN)
- new net LX1: L1.2, U3.3 (LX1)
- new net LX2: L1.1, U3.2 (LX2)
- no-connect marks 8 -> 6
Other:
- moved on the sheet: C1, C10, C13, C14, C2, C3, C4, C6, C7, D7, D8, D9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

Commit message: Before resize
Parts:
- U4: value TLV75512PDBV -> TLV75518PDBV
Changed lines of the file:
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@@
 			)
 		)
-		(property "Value" "TLV75512PDBV"
+		(property "Value" "TLV75518PDBV"
 			(at 95.25 22.86 0)
 			(effects
